File: template/Hammond_1593K_Enclosure/Hammond_1593K_Enclosure.kicad_sch (KiCad schematic)
At the start: 4 parts

Commit message: fix: change original libs; add: new components
- Fix LIS3DH pins positions;
- Add ATmega164P symbol;
- Add 3D model to the L_Wuerth_HCM-7050;
- Add parameters for R_RES (Assembly...).
- Add parameters for R_RES and C_CAP;
- Fix SOIC-8 package 3D model;
- Add new parameters for many symbols;
- Change text height from 70 mil to 50 mil;
- Add solder mask expansion for 2-contact jumpers;
- Change thermopad vias of QFN-20-1EP_3x3mm_P0.45mm_EP1.6x1.6mm_ThermalVias;
- Add D_SMAF footprint;
- Fillet silk for C_1206;
-Rectangle silk for R_1206;
Parts:
- removed MK1, MK2, MK3, MK4: Mounting_Hole, Mounting_Holes:MountingHole_3.2mm_M3_ISO7380, symbol Hammond_1593K_Enclosure:Mounting_Hole_PAD-Mechanical
Connections:
- no-connect marks 4 -> 0
Changed lines of the file:
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@@
-(kicad_sch (version 20210126) (generator eeschema)
+(kicad_sch (version 20211123) (generator eeschema)
   (paper "A4")
   (title_block
     (date "2021-02-16")
   )
-  (no_connect (at 106.68 185.42))
-  (no_connect (at 106.68 191.77))
-  (no_connect (at 129.54 185.42))
-  (no_connect (at 129.54 191.77))
-  (symbol (lib_id "Hammond_1593K_Enclosure:Mounting_Hole_PAD-Mechanical") (at 106.68 182.88 0) (unit 1)
-    (in_bom yes) (on_board yes)
-    (property "Reference" "MK1" (id 0) (at 109.22 181.7116 0)
-      (effects (font (size 1.27 1.27)) (justify left))
-    )
-    (property "Value" "Mounting_Hole" (id 1) (at 109.22 184.023 0)
-      (effects (font (size 1.27 1.27)) (justify left))
-    )
-    (property "Footprint" "Mounting_Holes:MountingHole_3.2mm_M3_ISO7380" (id 2) (at 106.68 182.88 0)
-      (effects (font (size 1.524 1.524)) hide)
-    )
-    (property "Datasheet" "" (id 3) (at 106.68 182.88 0)
-      (effects (font (size 1.524 1.524)) hide)
-    )
-    (pin "1")
-  )
-  (symbol (lib_id "Hammond_1593K_Enclosure:Mounting_Hole_PAD-Mechanical") (at 106.68 189.23 0) (unit 1)
-    (in_bom yes) (on_board yes)
-    (property "Reference" "MK2" (id 0) (at 109.22 188.0616 0)
-      (effects (font (size 1.27 1.27)) (justify left))
-    )
-    (property "Value" "Mounting_Hole" (id 1) (at 109.22 190.373 0)
-      (effects (font (size 1.27 1.27)) (justify left))
-    )
-    (property "Footprint" "Mounting_Holes:MountingHole_3.2mm_M3_ISO7380" (id 2) (at 106.68 189.23 0)
-      (effects (font (size 1.524 1.524)) hide)
-    )
-    (property "Datasheet" "" (id 3) (at 106.68 189.23 0)
-      (effects (font (size 1.524 1.524)) hide)
-    )
-    (pin "1")
-  )
-  (symbol (lib_id "Hammond_1593K_Enclosure:Mounting_Hole_PAD-Mechanical") (at 129.54 182.88 0) (unit 1)
-    (in_bom yes) (on_board yes)
-    (property "Reference" "MK3" (id 0) (at 132.08 181.7116 0)
-      (effects (font (size 1.27 1.27)) (justify left))
-    )
-    (property "Value" "Mounting_Hole" (id 1) (at 132.08 184.023 0)
-      (effects (font (size 1.27 1.27)) (justify left))
-    )
-    (property "Footprint" "Mounting_Holes:MountingHole_3.2mm_M3_ISO7380" (id 2) (at 129.54 182.88 0)
-      (effects (font (size 1.524 1.524)) hide)
-    )
-    (property "Datasheet" "" (id 3) (at 129.54 182.88 0)
-      (effects (font (size 1.524 1.524)) hide)
-    )
-    (pin "1")
-  )
-  (symbol (lib_id "Hammond_1593K_Enclosure:Mounting_Hole_PAD-Mechanical") (at 129.54 189.23 0) (unit 1)
-    (in_bom yes) (on_board yes)
-    (property "Reference" "MK4" (id 0) (at 132.08 188.0616 0)
-      (effects (font (size 1.27 1.27)) (justify left))
-    )
-    (property "Value" "Mounting_Hole" (id 1) (at 132.08 190.373 0)
-      (effects (font (size 1.27 1.27)) (justify left))
-    )
-    (property "Footprint" "Mounting_Holes:MountingHole_3.2mm_M3_ISO7380" (id 2) (at 129.54 189.23 0)
-      (effects (font (size 1.524 1.524)) hide)
-    )
-    (property "Datasheet" "" (id 3) (at 129.54 189.23 0)
-      (effects (font (size 1.524 1.524)) hide)
-    )
-    (pin "1")
-  )
   (sheet_instances
     (path "/" (page "1"))
   )
-  (symbol_instances
-    (path "/00000000-0000-0000-0000-00005867217e"
-      (reference "MK1") (unit 1) (value "Mounting_Hole") (footprint "Mounting_Holes:MountingHole_3.2mm_M3_ISO7380")
-    )
-    (path "/00000000-0000-0000-0000-0000586722b5"
-      (reference "MK2") (unit 1) (value "Mounting_Hole") (footprint "Mounting_Holes:MountingHole_3.2mm_M3_ISO7380")
-    )
-    (path "/00000000-0000-0000-0000-000058672295"
-      (reference "MK3") (unit 1) (value "Mounting_Hole") (footprint "Mounting_Holes:MountingHole_3.2mm_M3_ISO7380")
-    )
-    (path "/00000000-0000-0000-0000-00005867236d"
-      (reference "MK4") (unit 1) (value "Mounting_Hole") (footprint "Mounting_Holes:MountingHole_3.2mm_M3_ISO7380")
-    )
-  )
 )
